Commit message: added camera, friction, imu
+ added depth / rgb camera at gripper
+ added imu at gripper
+ added joint dynamics

File: arm_urdf/urdf/arm_desc.xacro (robot description, xacro)
@@ -4,18 +4,17 @@
     <xacro:property name="effort" value="30.0" />
     <xacro:property name="velocity" value="10.0" />
-    <xacro:macro name="default_inertial" params="mass">
-        <inertial>
-            <mass value="${mass}" />
-            <inertia ixx="1.0" ixy="0.0" ixz="0.0"
-                     iyy="1.0" iyz="0.0"
-                     izz="1.0" />
-        </inertial>
-    </xacro:macro>
-    <link name="base_footprint" />
+    <xacro:property name="damping" value="100" />
+    <xacro:property name="friction" value="100" />
+    <xacro:include filename="common.xacro"/>
+    <link name="base_footprint">
+        <xacro:inertial_box mass="10000" x="0.5" y="0.5" z="0.5">
+            <origin xyz="0 0 0.075" rpy="0 0 0"/>
+        </xacro:inertial_box>
+    </link>
     <link name="base_link">
         <xacro:default_inertial mass="1.0" />
         <visual>
             <geometry>
-                <mesh filename="package://arm_urdf/meshes/Base_Plate_.stl" scale="0.01 0.01 0.01" />
+                <mesh filename="file://$(find arm_urdf)/meshes/Base_Plate_.stl" scale="0.01 0.01 0.01" />
             </geometry>
             <origin xyz="0 0 0" rpy="${PI/2} 0 0" />
@@ -23,8 +22,11 @@
         <collision>
             <geometry>
-                <mesh filename="package://arm_urdf/meshes/Base_Plate_.stl" scale="0.01 0.01 0.01" />
+                <mesh filename="file://$(find arm_urdf)/meshes/Base_Plate_.stl" scale="0.01 0.01 0.01" />
             </geometry>
             <origin xyz="0 0 0" rpy="${PI/2} 0 0" />
         </collision>
+        <xacro:inertial_box mass="100" x="0.5" y="0.5" z="0.5">
+            <origin xyz="0 0 0.075" rpy="0 0 0"/>
+        </xacro:inertial_box>
     </link>
     <joint name="fixed_base_joint" type="fixed">
@@ -37,5 +39,5 @@
         <visual>
             <geometry>
-                <mesh filename="package://arm_urdf/meshes/Link1_.stl" scale="0.01 0.01 0.01" />
+                <mesh filename="file://$(find arm_urdf)/meshes/Link1_.stl" scale="0.01 0.01 0.01" />
             </geometry>
             <origin xyz="0 0 -0.508" rpy="${PI/2} 0 0" />
@@ -43,5 +45,5 @@
         <collision>
             <geometry>
-                <mesh filename="package://arm_urdf/meshes/Link1_.stl" scale="0.01 0.01 0.01" />
+                <mesh filename="file://$(find arm_urdf)/meshes/Link1_.stl" scale="0.01 0.01 0.01" />
             </geometry>
             <origin xyz="0 0 -0.508" rpy="${PI/2} 0 0" />
@@ -53,4 +55,6 @@
         <origin xyz="0 0 0.508" rpy="0 0 0" />
         <axis xyz="0 0 1" />
+        <limit lower="0" upper="${2*pi}" velocity="100" effort="100"/>
+        <dynamics damping="${damping}" friction="${friction}"/>
     </joint>
     <link name="link2">
@@ -58,5 +62,5 @@
         <visual>
             <geometry>
-                <mesh filename="package://arm_urdf/meshes/Link2_.stl" scale="0.01 0.01 0.01" />
+                <mesh filename="file://$(find arm_urdf)/meshes/Link2_.stl" scale="0.01 0.01 0.01" />
             </geometry>
             <origin xyz="0.098 0 -0.805" rpy="${PI/2} 0 0" />
@@ -64,5 +68,5 @@
         <collision>
             <geometry>
-                <mesh filename="package://arm_urdf/meshes/Link2_.stl" scale="0.01 0.01 0.01" />
+                <mesh filename="file://$(find arm_urdf)/meshes/Link2_.stl" scale="0.01 0.01 0.01" />
             </geometry>
             <origin xyz="0.098 0 -0.805" rpy="${PI/2} 0 0" />
@@ -74,4 +78,6 @@
         <origin xyz="-0.100 -0.01 0.300" rpy="0 0 0.08" />
         <axis xyz="0 1 0" />
+        <limit lower="0" upper="${2*pi}" velocity="100" effort="100"/>
+        <dynamics damping="${damping}" friction="${friction}"/>
     </joint>
     <link name="link3">
@@ -79,5 +85,5 @@
         <visual>
             <geometry>
-                <mesh filename="package://arm_urdf/meshes/Link3_.stl" scale="0.01 0.01 0.01" />
+                <mesh filename="file://$(find arm_urdf)/meshes/Link3_.stl" scale="0.01 0.01 0.01" />
             </geometry>
             <origin xyz="0.110 0 -3.15" rpy="${PI/2} 0 -0.02" />
@@ -85,5 +91,5 @@
         <collision>
             <geometry>
-                <mesh filename="package://arm_urdf/meshes/Link3_.stl" scale="0.01 0.01 0.01" />
+                <mesh filename="file://$(find arm_urdf)/meshes/Link3_.stl" scale="0.01 0.01 0.01" />
             </geometry>
             <origin xyz="0 0 0" rpy="0 0 0" />
@@ -95,4 +101,6 @@
         <origin xyz="-0.01 0 2.345" rpy="0 0 -0.05" />
         <axis xyz="0 1 0" />
+        <limit lower="0" upper="${2*pi}" velocity="100" effort="100"/>
+        <dynamics damping="${damping}" friction="${friction}"/>
     </joint>
     <link name="link4">
@@ -100,5 +108,5 @@
         <visual>
             <geometry>
-                <mesh filename="package://arm_urdf/meshes/Link4_.stl" scale="0.01 0.01 0.01" />
+                <mesh filename="file://$(find arm_urdf)/meshes/Link4_.stl" scale="0.01 0.01 0.01" />
             </geometry>
             <origin xyz="0.098 0 -5.32" rpy="${PI/2} 0 0" />
@@ -106,5 +114,5 @@
         <collision>
             <geometry>
-                <mesh filename="package://arm_urdf/meshes/Link4_.stl" scale="0.01 0.01 0.01" />
+                <mesh filename="file://$(find arm_urdf)/meshes/Link4_.stl" scale="0.01 0.01 0.01" />
             </geometry>
             <origin xyz="0 0 0" rpy="0 0 0" />
@@ -116,4 +124,6 @@
         <origin xyz="0 -0.0055 2.168" rpy="0 0 0.05" />
         <axis xyz="0 1 0" />
+        <limit lower="0" upper="${2*pi}" velocity="100" effort="100"/>
+        <dynamics damping="${damping}" friction="${friction}"/>
     </joint>
     <link name="link5">
@@ -121,5 +131,5 @@
         <visual>
             <geometry>
-                <mesh filename="package://arm_urdf/meshes/Link5_.stl" scale="0.01 0.01 0.01" />
+                <mesh filename="file://$(find arm_urdf)/meshes/Link5_.stl" scale="0.01 0.01 0.01" />
             </geometry>
             <origin xyz="0.098 0 -7.574" rpy="${PI/2} 0 0" />
@@ -127,5 +137,5 @@
         <collision>
             <geometry>
-                <mesh filename="package://arm_urdf/meshes/Link5_.stl" scale="0.01 0.01 0.01" />
+                <mesh filename="file://$(find arm_urdf)/meshes/Link5_.stl" scale="0.01 0.01 0.01" />
             </geometry>
             <origin xyz="0 0 0" rpy="0 0 0" />
@@ -137,4 +147,6 @@
         <origin xyz="0 0 2.253" rpy="0 0 0" />
         <axis xyz="0 1 0" />
+        <limit lower="0" upper="${2*pi}" velocity="100" effort="100"/>
+        <dynamics damping="${damping}" friction="${friction}"/>
     </joint>
     <link name="gripper">
@@ -142,5 +154,5 @@
         <visual>
             <geometry>
-                <mesh filename="package://arm_urdf/meshes/Link6_.stl" scale="0.01 0.01 0.01" />
+                <mesh filename="file://$(find arm_urdf)/meshes/Link6_.stl" scale="0.01 0.01 0.01" />
             </geometry>
             <origin xyz="0.09 0.022 -8.285" rpy="${PI/2} 0 0" />
@@ -148,5 +160,5 @@
         <collision>
             <geometry>
-                <mesh filename="package://arm_urdf/meshes/Link6_.stl" scale="0.01 0.01 0.01" />
+                <mesh filename="file://$(find arm_urdf)/meshes/Link6_.stl" scale="0.01 0.01 0.01" />
             </geometry>
             <origin xyz="0 0 0" rpy="0 0 0" />
@@ -158,4 +170,43 @@
         <origin xyz="0.01 -0.033 0.72" rpy="0 0 0" />
         <axis xyz="0 0 1" />
-    </joint>
+        <limit lower="0" upper="${2*pi}" velocity="100" effort="100"/>
+        <dynamics damping="${damping}" friction="${friction}"/>
+    </joint>
+    <joint name="gripper_camera_joint" type="fixed">
+        <origin xyz="-0.3 0 1.5" rpy="0 ${PI/-2} 0"/>
+        <parent link="gripper"/>
+        <child link="camera"/>
+    </joint>
+    <link name="camera">
+        <visual>
+            <origin xyz="0 0 0" rpy="0 0 0"/>
+            <geometry>
+                <box size="0.06 0.15 0.15" />
+            </geometry>
+            <material name="green" />
+        </visual>
+        <visual>
+            <origin xyz="0.03 0 0" rpy="0 ${pi/2} 0"/>
+            <geometry>
+                <cylinder length="0.06" radius="0.04" />
+            </geometry>
+            <material name="blue" />
+        </visual>
+        <collision>
+            <origin xyz="0.0 0 0" rpy="0 0 0"/>
+            <geometry>
+                <box size="0.12 0.15 0.15" />
+            </geometry>
+        </collision>
+        <xacro:inertial_box mass="0.1" x="0.12" y="0.15" z="0.15">
+            <origin xyz="0.0 0 0" rpy="0 0 0"/>
+        </xacro:inertial_box>
+    </link>
+    <joint name="camera_optical_joint" type="fixed">
+        <origin xyz="0.13 0 0" rpy="0 0 0" />
+        <parent link="camera" />
+        <child link="camera_link_optical" />
+    </joint>
+    <link name="camera_link_optical"/>
+    <xacro:include filename="gazebo.xacro"/>
 </robot>
